File: cgb-reg/CBG-REG.kicad_sch (KiCad schematic)
At the start: 49 parts, among them J1 Conn_01x07, J2 Conn_01x07, U3 GS8624-SR, U4 74LVC2G04, U5 GS8624-SR, U6 GS8624-SR

Commit message: feat: Add v1.0 of power distribution board
also slight reorg of repo
Parts:
- J1, J2: now left out of the parts list
Changed lines of the file:
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@@
   )
   (symbol (lib_id "Connector_Generic:Conn_01x07") (at 29.21 176.53 0) (mirror y) (unit 1)
-    (in_bom yes) (on_board yes) (dnp no)
+    (in_bom no) (on_board yes) (dnp no)
     (property "Reference" "J1" (at 29.21 166.37 0)
       (effects (font (size 1.27 1.27)))
@@
   )
   (symbol (lib_id "Connector_Generic:Conn_01x07") (at 55.88 176.53 180) (unit 1)
-    (in_bom yes) (on_board yes) (dnp no)
+    (in_bom no) (on_board yes) (dnp no)
     (property "Reference" "J2" (at 55.88 166.37 0)
       (effects (font (size 1.27 1.27)))
