File: cgb-reg/CGB-REG.kicad_pcb (KiCad board)
At the start: 2 copper layers, 31 x 26.5 mm, 50 parts, among them J1 Conn_01x07, J2 Conn_01x07, U3 GS8624-SR, U4 74LVC2G04, U5 GS8624-SR, U6 GS8624-SR

Commit message: fix: Fix wrong footprint for inverter IC
Parts:
- U4: footprint Package_TO_SOT_SMD:SOT-23-6 -> Package_TO_SOT_SMD:SOT-363_SC-70-6
Routing:
- net +5V: track 26.5 -> 27.4 mm
- net 'SW: track 40.8 -> 40.0 mm
Other:
- board text added: "V1.2"
- board text removed: "V1.1"
