File: cgb-reg/CGB-REG.kicad_sch (KiCad schematic)
At the start: 49 parts, among them J1 Conn_01x07, J2 Conn_01x07, U3 GS8624-SR, U4 74LVC2G04, U5 GS8624-SR, U6 GS8624-SR

Commit message: fix: Fix wrong footprint for inverter IC
Parts:
- U4: footprint Package_TO_SOT_SMD:SOT-23-6 -> Package_TO_SOT_SMD:SOT-363_SC-70-6
