File: pwr-dist/pwr-dist.kicad_pcb (KiCad board)
At the start: 2 copper layers, 22.2 x 23.2 mm, 24 parts, among them J1 Conn_01x04, J2 Conn_01x06, Q1 2SA1576AT, Q2 UMZ2NTR, Q3 BSD235C

Commit message: feat: Add a new breakout for the official CGB-REG IC
Parts:
- J1, J2: moved to B.Cu
- turned J1 to 180 degrees
- turned J2 to 180 degrees
